Commit message: update models

File: src/nana_v3_description/assets/robot/urdf/nana_v3.urdf (robot description, URDF)
Before this commit: robot openarm, 20 links, 19 joints
Joints:
- joint nana_v3_left_nana_v3_body_link0_joint: origin xyz=0.0 0.031 0.698 rpy=-1.5708 0 0 -> xyz=0.0 0.18 1.22 rpy=-1.5708 0 0
- joint nana_v3_right_nana_v3_body_link0_joint: origin xyz=0.0 -0.031 0.698 rpy=1.5708 0 0 -> xyz=0.0 -0.18 1.22 rpy=1.5708 0 0

File: src/nana_v3_description/assets/robot/urdf/nana_v3_corrected.urdf (robot description, URDF)
Before this commit: robot openarm, 20 links, 19 joints
Links:
- link nana_v3_left_hand: mass 0.1  -> 0.1
- link nana_v3_left_link0: mass 1.1432284943239561 -> 1.143228
- link nana_v3_left_link1: mass 1.1416684646202298 -> 1.141668
- link nana_v3_left_link2: mass 0.2775092746011571 -> 0.277509
- link nana_v3_left_link3: mass 1.073863338202347 -> 1.073863
- link nana_v3_left_link4: mass 0.6348534566833373 -> 0.634853
- link nana_v3_left_link5: mass 0.6156588026168502 -> 0.615659
- link nana_v3_left_link6: mass 0.475202773187987 -> 0.475203
- link nana_v3_left_link7: mass 0.4659771327380578 -> 0.465977
- link nana_v3_right_link0: mass 1.1432284943239561 -> 1.143228
- link nana_v3_right_link1: mass 1.1416684646202298 -> 1.141668
- link nana_v3_right_link2: mass 0.2775092746011571 -> 0.277509
- link nana_v3_right_link3: mass 1.073863338202347 -> 1.073863
- link nana_v3_right_link4: mass 0.6348534566833373 -> 0.634853
- link nana_v3_right_link5: mass 0.6156588026168502 -> 0.615659
- link nana_v3_right_link6: mass 0.475202773187987 -> 0.475203
- link nana_v3_right_link7: mass 0.4659771327380578 -> 0.465977
Joints:
- removed joint nana_v3_left_joint3
- joint nana_v3_left_joint2: origin xyz=-0.0301 0.0 0.06 rpy=-1.57079632679 0 0 -> xyz=-0.0301 0.0 0.06 rpy=-1.570796 0 0
- joint nana_v3_left_joint4: origin xyz=-0.0 0.0315 0.15375 rpy=0 0 0 -> xyz=0.0 0.0315 0.15375 rpy=0 0 0
- joint nana_v3_right_joint2: origin xyz=-0.0301 0.0 0.06 rpy=1.57079632679 0 0 -> xyz=-0.0301 0.0 0.06 rpy=1.570796 0 0
- joint nana_v3_right_joint4: origin xyz=-0.0 0.0315 0.15375 rpy=0 0 0 -> xyz=0.0 0.0315 0.15375 rpy=0 0 0
